File: digital-clock-pcb/digital-clock.kicad_pcb (KiCad board)
At the start: 2 copper layers, 50 x 100 mm, 29 parts, among them J1 USB_OTG, J2 Conn_02x03_Odd_Even, U1 ATmega328P-M, U2 PCF8523T, Y1 ABS2532768KHZ6T

Commit message: update silkscreen
Parts:
- moved D1 2.00 mm to (115.0, 95.4), turned to -90 degrees
- moved D11 2.00 mm to (115.3, 74.1)
- moved D13 2.00 mm to (155.0, 95.7)
- moved D3 2.00 mm to (155.0, 74.5)
- moved D6 2.00 mm to (115.2, 84.5)
- moved D8 2.00 mm to (155.0, 84.5)
Connections:
- U1 pad 13: unconnected-(U1-Pad13) -> WS_IN
- U1 pad 18: unconnected-(U1-Pad18) -> VCC
- U1 pad 21: Net-(U1-Pad21) -> GND
- U1 pad 27: unconnected-(U1-Pad27) -> SDA
- U1 pad 28: unconnected-(U1-Pad28) -> SCL
- U1 pad 29: unconnected-(U1-Pad29) -> RST
- U1 pad 3: Net-(U1-Pad21) -> GND
- U1 pad 33: Net-(U1-Pad21) -> GND
- U1 pad 4: Net-(U1-Pad4) -> VCC
- U1 pad 5: Net-(U1-Pad21) -> GND
- U1 pad 6: Net-(U1-Pad4) -> VCC
Routing:
- net VCC: track 6.88 -> 310.3 mm, vias 0 -> 3
- net WS_IN: track 0.00 -> 26.9 mm, vias 0 -> 1
- net RST: track 0.00 -> 23.3 mm, vias 0 -> 1
- net SCL: track 5.42 -> 24.4 mm
- net Net-(D14-Pad4): track 0.00 -> 17.0 mm
- net Net-(D14-Pad2): track 0.00 -> 16.1 mm
- net Net-(D13-Pad2): track 0.00 -> 15.8 mm
- net Net-(U2-Pad1): track 0.00 -> 12.8 mm
- net Net-(D17-Pad4): track 0.00 -> 11.6 mm
- net Net-(D2-Pad4): track 0.00 -> 11.5 mm
- net Net-(D3-Pad4): track 0.00 -> 11.4 mm
- net SDA: track 3.23 -> 14.5 mm
- net Net-(D15-Pad2): track 0.00 -> 11.1 mm
- net SCK: track 0.00 -> 8.94 mm
- net Net-(D13-Pad4): track 0.00 -> 7.63 mm
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- added copper zone on B.Cu, net GND
- added copper zone on F.Cu, net GND

Commit message: wiring connector
Parts:
- added J3: OUT, Connector_JST:JST_SH_SM04B-SRSS-TB_1x04-1MP_P1.00mm_Horizontal, F.Cu at (117.1, 66.8)
- added J4: IN, Connector_JST:JST_SH_SM04B-SRSS-TB_1x04-1MP_P1.00mm_Horizontal, F.Cu at (153.3, 67.0)
Connections:
- D21 pad 2: unconnected-(D21-Pad2) -> WS_OUT
Routing:
- net WS_OUT: track 0.00 -> 108.1 mm, vias 0 -> 1
- net WS_IN: track 26.9 -> 98.4 mm, vias 1 -> 2
- net VCC: track 310.3 -> 324.8 mm, vias 3 -> 5
- net GND: vias 10 -> 17
