File: digital-clock-pcb/digital-clock.kicad_sch (KiCad schematic)
At the start: 31 parts, among them J1 USB_OTG, J2 Conn_02x03_Odd_Even, J3 Conn_01x04, J4 Conn_01x04, U1 ATmega328P-M, U2 PCF8523T, Y1 ABS2532768KHZ6T

Commit message: change m328 package
Parts:
- U1: footprint Package_DFN_QFN:QFN-32-1EP_5x5mm_P0.5mm_EP3.1x3.1mm -> Package_QFP:TQFP-32_7x7mm_P0.8mm
Changed lines of the file:
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@@
       (effects (font (size 1.27 1.27)) (justify left))
     )
-    (property "Footprint" "Package_DFN_QFN:QFN-32-1EP_5x5mm_P0.5mm_EP3.1x3.1mm" (id 2) (at 35.56 99.06 0)
+    (property "Footprint" "Package_QFP:TQFP-32_7x7mm_P0.8mm" (id 2) (at 35.56 99.06 0)
       (effects (font (size 1.27 1.27) italic) hide)
     )
@@
     )
     (path "/ebd1509e-daba-42cf-8f1c-294b259f2169"
-      (reference "U1") (unit 1) (value "ATmega328P-M") (footprint "Package_DFN_QFN:QFN-32-1EP_5x5mm_P0.5mm_EP3.1x3.1mm")
+      (reference "U1") (unit 1) (value "ATmega328P-M") (footprint "Package_QFP:TQFP-32_7x7mm_P0.8mm")
     )
     (path "/d7af507e-f887-4995-925b-7c5f77d83df7"

Commit message: add clock battery + add button for change hour and minute
Parts:
- added BT1: Battery_Cell, Battery:BatteryHolder_LINX_BAT-HLD-012-SMT, symbol Device:Battery_Cell
- added R3, R4: R_Small, Resistor_SMD:R_0603_1608Metric, symbol Device:R_Small
- added SW1, SW2: SW_SPST, Button_Switch_SMD:SW_SPST_FSMSM, symbol Switch:SW_SPST
Connections:
- net GND: now also BT1.2 (-), R3.2, R4.2
- net VCC: now also SW1.1 (A), SW2.1 (A)
- net at U2.3 (VBAT): now also BT1.1 (+)
- net BTN1: now reaches U1.23 (PC0)
- net BTN1: now also R4.1, SW1.2 (B)
- net BTN2: now reaches U1.24 (PC1)
- net BTN2: now also R3.1, SW2.2 (B)
